Commit message: fix dobot robot URDF and pybullet setup

File: data/dobot/dobot.urdf (robot description, URDF)
Before this commit: robot urdf_door, 10 links, 9 joints
Links:
- link linkC: geometry collision box size=0.026 0.026 0.21; visual mesh filename=cad/Dobot/A6_7.stl scale=1 1 1
- link linkD: geometry collision box size=0.02 0.08 0.005; visual mesh filename=cad/Dobot/A16.stl scale=1 1 1
- link motorA: geometry collision cylinder length=0.03 radius=0.02; visual cylinder length=0.03 radius=0.02
- link motorB: geometry collision cylinder length=0.03 radius=0.02; visual cylinder length=0.03 radius=0.02
Joints:
- joint joint_linkAlinkA9: origin xyz=0 -0.035 0.045 -> xyz=0 -0.026 0.054
