Commit message: add Wavefront obj files for ANYmal (allows for caching and using p.loadURDF flag anymal = p.loadURDF("ANYmal/robot.urdf",[i*1,j*1,0.6], flags=p.URDF_ENABLE_CACHED_GRAPHICS_SHAPES)

File: data/ANYmal/robot.urdf (robot description, URDF)
Before this commit: robot anymal, 18 links, 17 joints
Links:
- link LF_FOOT_MOUNT: geometry collision sphere radius=0.03; visual mesh filename=anymal_optoforce.obj scale=0.001 0.001 0.001
- link LF_SHANK: geometry collision cylinder length=0.19 radius=0.015; visual mesh filename=anymal_shank_2_LF.obj scale=0.001 0.001 0.001
- link LF_THIGH: geometry collision cylinder length=0.08 radius=0.04; visual mesh filename=anymal_thigh.obj scale=0.001 0.001 0.001
- link LH_FOOT_MOUNT: geometry collision sphere radius=0.03; visual mesh filename=anymal_optoforce.obj scale=0.001 0.001 0.001
- link LH_SHANK: geometry collision cylinder length=0.19 radius=0.015; visual mesh filename=anymal_shank_2_LH.obj scale=0.001 0.001 0.001
- link LH_THIGH: geometry collision cylinder length=0.08 radius=0.04; visual mesh filename=anymal_thigh.obj scale=0.001 0.001 0.001
- link RF_FOOT_MOUNT: geometry collision sphere radius=0.03; visual mesh filename=anymal_optoforce.obj scale=0.001 0.001 0.001
- link RF_SHANK: geometry collision cylinder length=0.19 radius=0.015; visual mesh filename=anymal_shank_2_RF.obj scale=0.001 0.001 0.001
- link RF_THIGH: geometry collision cylinder length=0.08 radius=0.04; visual mesh filename=anymal_thigh.obj scale=0.001 0.001 0.001
- link RH_FOOT_MOUNT: geometry collision sphere radius=0.03; visual mesh filename=anymal_optoforce.obj scale=0.001 0.001 0.001
- link RH_SHANK: geometry collision cylinder length=0.19 radius=0.015; visual mesh filename=anymal_shank_2_RH.obj scale=0.001 0.001 0.001
- link RH_THIGH: geometry collision cylinder length=0.08 radius=0.04; visual mesh filename=anymal_thigh.obj scale=0.001 0.001 0.001
