Commit message: fix relative path for franka

File: data/franka_panda/panda.urdf (robot description, URDF)
Before this commit: robot panda, 12 links, 11 joints
Links:
- link panda_hand: geometry collision mesh filename=package://meshes/collision/hand.obj; visual mesh filename=package://meshes/collision/hand.obj
- link panda_leftfinger: geometry collision mesh filename=package://meshes/collision/finger.obj; visual mesh filename=package://meshes/collision/finger.obj
- link panda_link0: geometry collision mesh filename=package://meshes/collision/link0.obj; visual mesh filename=package://meshes/collision/link0.obj
- link panda_link1: geometry collision mesh filename=package://meshes/collision/link1.obj; visual mesh filename=package://meshes/collision/link1.obj
- link panda_link2: geometry collision mesh filename=package://meshes/collision/link2.obj; visual mesh filename=package://meshes/collision/link2.obj
- link panda_link3: geometry collision mesh filename=package://meshes/collision/link3.obj; visual mesh filename=package://meshes/collision/link3.obj
- link panda_link4: geometry collision mesh filename=package://meshes/collision/link4.obj; visual mesh filename=package://meshes/collision/link4.obj
- link panda_link5: geometry collision mesh filename=package://meshes/collision/link5.obj; visual mesh filename=package://meshes/collision/link5.obj
- link panda_link6: geometry collision mesh filename=package://meshes/collision/link6.obj; visual mesh filename=package://meshes/collision/link6.obj
- link panda_link7: geometry collision mesh filename=package://meshes/collision/link7.obj; visual mesh filename=package://meshes/collision/link7.obj
- link panda_rightfinger: geometry collision mesh filename=package://meshes/collision/finger.obj; visual mesh filename=package://meshes/collision/finger.obj

Commit message: Add Franka Panda Emika example, improve assets

File: data/franka_panda/panda.urdf (robot description, URDF)
Before this commit: robot panda, 12 links, 11 joints
Links:
- link panda_hand: geometry collision mesh filename=package://meshes/collision/hand.obj; visual mesh filename=package://meshes/visual/hand.obj
- link panda_leftfinger: geometry collision mesh filename=package://meshes/collision/finger.obj; visual mesh filename=package://meshes/visual/finger.obj
- link panda_link1: geometry collision mesh filename=package://meshes/collision/link1.obj; visual mesh filename=package://meshes/visual/link1.obj
- link panda_link2: geometry collision mesh filename=package://meshes/collision/link2.obj; visual mesh filename=package://meshes/visual/link2.obj
- link panda_link3: geometry collision mesh filename=package://meshes/collision/link3.obj; visual mesh filename=package://meshes/visual/link3.obj
- link panda_link4: geometry collision mesh filename=package://meshes/collision/link4.obj; visual mesh filename=package://meshes/visual/link4.obj
- link panda_link5: geometry collision mesh filename=package://meshes/collision/link5.obj; visual mesh filename=package://meshes/visual/link5.obj
- link panda_link6: geometry collision mesh filename=package://meshes/collision/link6.obj; visual mesh filename=package://meshes/visual/link6.obj
- link panda_rightfinger: geometry collision mesh filename=package://meshes/collision/finger.obj; visual mesh filename=package://meshes/visual/finger.obj

Commit message: add IK to loadpanda.py example add estimated masses and center of mass to Franka Panda (sums up to 18kg)

File: data/franka_panda/panda.urdf (robot description, URDF)
Before this commit: robot panda, 12 links, 11 joints
Links:
- link panda_hand: mass None -> .81
- link panda_leftfinger: mass None -> 0.1
- link panda_link0: mass None -> 2.9
- link panda_link1: mass None -> 2.7
- link panda_link2: mass None -> 2.73
- link panda_link3: mass None -> 2.04
- link panda_link4: mass None -> 2.08
- link panda_link5: mass None -> 3
- link panda_link6: mass None -> 1.3
- link panda_link7: mass None -> .2
- link panda_rightfinger: mass None -> 0.1

Commit message: improved version of panda sim benchmark

File: data/franka_panda/panda.urdf (robot description, URDF)
Before this commit: robot panda, 12 links, 11 joints
Links:
- added link panda_grasptarget, mass 0.0
- link panda_link8: mass None -> 0.0
Joints:
- added joint panda_grasptarget_hand: type fixed, parent panda_hand, child panda_grasptarget, origin xyz=0 0 0.105 rpy=0 0 0
