Commit message: update Laikago model with textures, add version with toes for inverse kinematics, fix mass of hip motors (from 1kg -> 0.241kg)

File: data/laikago/laikago.urdf (robot description, URDF)
Before this commit: robot plane, 13 links, 12 joints
Links:
- link FL_hip_motor: geometry collision mesh filename=hip_motor.stl scale=1 1 1; visual mesh filename=hip_motor.obj scale=1 1 1
- link FL_lower_leg: geometry collision mesh filename=lower_leg_3_collision.stl scale=1 1 1; visual mesh filename=lower_leg3.obj scale=1 1 1
- link FL_upper_leg: geometry collision mesh filename=upper_leg_left_vhacd.obj scale=1 1 1; visual mesh filename=upper_leg_left.obj scale=1 1 1
- link FR_hip_motor: mass 1.095 -> 0.241; geometry collision mesh filename=hip_motor_mirror.stl scale=1 1 1; visual mesh filename=hip_motor_mirror.obj scale=1 1 1
- link FR_lower_leg: geometry collision mesh filename=lower_leg_3_collision.stl scale=1 1 1; visual mesh filename=lower_leg3.obj scale=1 1 1
- link FR_upper_leg: geometry collision mesh filename=upper_leg_right_vhacd.obj scale=1 1 1; visual mesh filename=upper_leg_mirror.obj scale=1 1 1
- link RL_hip_motor: geometry collision mesh filename=hip_motor.stl scale=1 1 1; visual mesh filename=hip_motor.obj scale=1 1 1
- link RL_lower_leg: geometry collision mesh filename=lower_leg_3_collision.stl scale=1 1 1; visual mesh filename=lower_leg3.obj scale=1 1 1
- link RL_upper_leg: geometry collision mesh filename=upper_leg_left_vhacd.obj scale=1 1 1; visual mesh filename=upper_leg_left2.obj scale=1 1 1
- link RR_hip_motor: mass 1.095 -> 0.241; geometry collision mesh filename=hip_motor_mirror.stl scale=1 1 1; visual mesh filename=hip_motor_mirror.obj scale=1 1 1
- link RR_lower_leg: geometry collision mesh filename=lower_leg_3_collision.stl scale=1 1 1; visual mesh filename=lower_leg3.obj scale=1 1 1
- link RR_upper_leg: geometry collision mesh filename=upper_leg_right_vhacd.obj scale=1 1 1; visual mesh filename=upper_leg_mirror2.obj scale=1 1 1
- link chassis: geometry collision mesh filename=chassis_vhacd_mod.obj scale=1 1 1; visual mesh filename=chassis.obj scale=1 1 1

Commit message: fix issue with hip motor mass in previous commit

File: data/laikago/laikago.urdf (robot description, URDF)
Before this commit: robot plane, 13 links, 12 joints
Links:
- link FR_hip_motor: mass 0.241 -> 1.095
- link RR_hip_motor: mass 0.241 -> 1.095
